File: rings/rings_panel/rings.kicad_pcb (KiCad board)
At the start: 2 copper layers, 70.8 x 128.5 mm, 24 parts

Commit message: Add files via upload
Fixed a small issue on the front panel
Parts:
- removed the G*** at (0.00, 0.00)
Changed lines of the file:
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@@
       ) (layer "B.Cu") (width 0.01) (fill solid))
-  )
-  (footprint "LOGO" (layer "F.Cu")
-    (at 0 0)
-    (attr through_hole)
-    (fp_text reference "G***" (at 0 0) (layer "F.SilkS") hide
-      (effects (font (size 1.524 1.524) (thickness 0.3)))
-    )
-    (fp_text value "LOGO" (at 0.75 0) (layer "F.SilkS") hide
-      (effects (font (size 1.524 1.524) (thickness 0.3)))
-    )
-    (fp_poly (pts
-        (xy -18.79162 61.776378)
-        (xy -18.716745 61.803906)
-        (xy -18.621312 61.873725)
-        (xy -18.555904 61.965107)
-        (xy -18.520607 62.069928)
-        (xy -18.515506 62.180064)
-        (xy -18.540686 62.287393)
-        (xy -18.596234 62.383791)
-        (xy -18.682235 62.461134)
-        (xy -18.709645 62.477147)
-        (xy -18.817057 62.515343)
-        (xy -18.930113 62.524253)
-        (xy -19.033671 62.503277)
-        (xy -19.060583 62.491086)
-        (xy -19.146012 62.436894)
-        (xy -19.204405 62.373976)
-        (xy -19.243024 62.304083)
-        (xy -19.276099 62.184711)
-        (xy -19.269932 62.064809)
-        (xy -19.226663 61.952789)
-        (xy -19.14843 61.85706)
-        (xy -19.124318 61.83716)
-        (xy -19.024411 61.785672)
-        (xy -18.908709 61.765019)
-        (xy -18.79162 61.776378)
-      ) (layer "F.Mask") (width 0.01) (fill solid))
-    (fp_poly (pts
-        (xy -17.513823 58.535131)
-        (xy -17.409429 58.594724)
-        (xy -17.397702 58.604257)
-        (xy -17.317748 58.695184)
-        (xy -17.27493 58.804034)
-        (xy -17.265952 58.896788)
-        (xy -17.284679 59.024108)
-        (xy -17.338544 59.130036)
-        (xy -17.424078 59.210538)
-        (xy -17.537808 59.261581)
-        (xy -17.5895 59.272702)
-        (xy -17.645014 59.278741)
-        (xy -17.682429 59.277991)
-        (xy -17.68475 59.277382)
-        (xy -17.719941 59.267876)
-        (xy -17.763737 59.257629)
-        (xy -17.838634 59.22355)
-        (xy -17.913074 59.160488)
-        (xy -17.975051 59.080187)
-        (xy -18.003412 59.023152)
-        (xy -18.029363 58.905388)
-        (xy -18.018938 58.795905)
-        (xy -17.977875 58.698672)
-        (xy -17.911913 58.617657)
-        (xy -17.826789 58.556827)
-        (xy -17.728241 58.52015)
-        (xy -17.622006 58.511596)
-        (xy -17.513823 58.535131)
-      ) (layer "F.Mask") (width 0.01) (fill solid))
-    (fp_poly (pts
-        (xy -19.987405 58.54893)
-        (xy -19.887545 58.611821)
-        (xy -19.81231 58.697304)
-        (xy -19.800656 58.717803)
-        (xy -19.779284 58.788236)
-        (xy -19.77067 58.880117)
-        (xy -19.775301 58.974379)
-        (xy -19.792243 59.04833)
-        (xy -19.8498 59.144077)
-        (xy -19.936187 59.217422)
-        (xy -20.041681 59.263444)
-        (xy -20.156556 59.277223)
-        (xy -20.226218 59.2679)
-        (xy -20.345446 59.219754)
-        (xy -20.438561 59.141129)
-        (xy -20.500954 59.037225)
-        (xy -20.526812 58.928744)
-        (xy -20.518616 58.807598)
-        (xy -20.473995 58.697628)
-        (xy -20.398701 58.606403)
-        (xy -20.298488 58.541491)
-        (xy -20.212245 58.51495)
-        (xy -20.099702 58.514636)
-        (xy -19.987405 58.54893)
-      ) (layer "F.Mask") (width 0.01) (fill solid))
-    (fp_poly (pts
-        (xy -19.97539 61.804254)
-        (xy -19.959447 61.811958)
-        (xy -19.868686 61.879109)
-        (xy -19.80678 61.968735)
-        (xy -19.77364 62.07242)
-        (xy -19.769175 62.181746)
-        (xy -19.793298 62.288297)
-        (xy -19.845918 62.383655)
-        (xy -19.926947 62.459402)
-        (xy -19.96655 62.481967)
-        (xy -20.073201 62.516549)
-        (xy -20.184525 62.524067)
-        (xy -20.284702 62.504012)
-        (xy -20.309369 62.492987)
-        (xy -20.396824 62.436756)
-        (xy -20.457331 62.368088)
-        (xy -20.491858 62.304083)
-        (xy -20.526638 62.184135)
-        (xy -20.519308 62.065343)
-        (xy -20.491661 61.986583)
-        (xy -20.421807 61.88007)
-        (xy -20.329225 61.806603)
-        (xy -20.219944 61.76816)
-        (xy -20.099989 61.766718)
-        (xy -19.97539 61.804254)
-      ) (layer "F.Mask") (width 0.01) (fill solid))
-    (fp_poly (pts
-        (xy -17.557104 61.774397)
-        (xy -17.450826 61.812346)
-        (xy -17.363157 61.878322)
-        (xy -17.338103 61.908845)
-        (xy -17.286043 62.016335)
-        (xy -17.267399 62.137326)
-        (xy -17.282134 62.259378)
-        (xy -17.33021 62.370047)
-        (xy -17.339518 62.383809)
-        (xy -17.415067 62.455811)
-        (xy -17.514725 62.502857)
-        (xy -17.626892 62.522729)
-        (xy -17.739968 62.513209)
-        (xy -17.832291 62.478038)
-        (xy -17.928715 62.401651)
-        (xy -17.992964 62.305009)
-        (xy -18.024441 62.196051)
-        (xy -18.022548 62.082719)
-        (xy -17.986685 61.972953)
-        (xy -17.916255 61.874695)
-        (xy -17.880217 61.841956)
-        (xy -17.782538 61.787877)
-        (xy -17.671255 61.765798)
-        (xy -17.557104 61.774397)
-      ) (layer "F.Mask") (width 0.01) (fill solid))
-    (fp_poly (pts
-        (xy -18.817615 60.272767)
-        (xy -18.718814 60.305335)
-        (xy -18.624462 60.372078)
-        (xy -18.559201 60.461395)
-        (xy -18.523112 60.565032)
-        (xy -18.516274 60.674736)
-        (xy -18.538767 60.782251)
-        (xy -18.590672 60.879324)
-        (xy -18.672067 60.957699)
-        (xy -18.712272 60.981646)
-        (xy -18.810434 61.013331)
-        (xy -18.922223 61.021575)
-        (xy -19.027484 61.005685)
-        (xy -19.060583 60.99362)
-        (xy -19.149366 60.932932)
-        (xy -19.22104 60.843373)
-        (xy -19.267867 60.737357)
-        (xy -19.282368 60.637888)
-        (xy -19.269181 60.558422)
-        (xy -19.236146 60.470889)
-        (xy -19.191669 60.394713)
-        (xy -19.16334 60.362849)
-        (xy -19.060185 60.29814)
-        (xy -18.941269 60.267637)
-        (xy -18.817615 60.272767)
-      ) (layer "F.Mask") (width 0.01) (fill solid))
   )
   (footprint "Wire_Pads:SolderWirePad_single_0-8mmDrill" (layer "F.Cu")
